File: hardware/ZSWatch-Dock.kicad_pcb (KiCad board)
At the start: 4 copper layers, 80 x 48 mm, 75 parts, among them IC101 TLV70218_SOT23-5, IC102 USBLC6-2P6, IC103 FT230XQ, IC104 MIC5219-3.3YM5, IC105 NL3V4T244MU2TAG-Q, IC106 USBLC6-2P6, IC107 USB2512BT, IC108 USBLC6-2P6, IC109 MIC2026-1xM, J102 Voltage, Q101 BSH205G2AR, SW101 Charge, X101 Debug, X102 UART, X103 Host, X104 Device, X105 Current, Y101 24 MHz

Commit message: Issue #42
Parts:
- removed the REF** at (129.0, 139.0)
- removed the REF** at (201.0, 139.0)
- removed the REF** at (201.0, 99.0)
- removed the REF** at (129.0, 99.0)
- added REF**: MountingHole_3.2mm_M3_Pad_Via, MountingHole:MountingHole_3.2mm_M3_Pad_Via, F.Cu at (243.7, 167.1)
- added REF**: MountingHole_3.2mm_M3_Pad_Via, MountingHole:MountingHole_3.2mm_M3_Pad_Via, F.Cu at (243.7, 127.1)
- added REF**: MountingHole_3.2mm_M3_Pad_Via, MountingHole:MountingHole_3.2mm_M3_Pad_Via, F.Cu at (171.7, 167.1)
- added REF**: MountingHole_3.2mm_M3_Pad_Via, MountingHole:MountingHole_3.2mm_M3_Pad_Via, F.Cu at (171.7, 127.1)
- moved C106 51.1 mm to (203.9, 151.2)
- moved C108 51.1 mm to (223.9, 135.8)
- moved C116 51.1 mm to (216.0, 142.7)
- moved C118 51.1 mm to (212.2, 144.9)
- moved IC102 51.1 mm to (198.4, 130.7)
- moved IC105 51.1 mm to (192.4, 128.9)
- moved IC106 51.1 mm to (235.8, 148.5)
- moved R103 51.1 mm to (191.1, 125.2)
- moved R105 51.1 mm to (241.4, 142.1)
- moved R106 51.1 mm to (239.3, 154.6)
- moved R111 51.1 mm to (217.3, 152.3)
- moved SB101 51.1 mm to (192.4, 126.0)
- moved SB102 51.1 mm to (192.4, 128.6)
- moved SB103 51.1 mm to (192.4, 131.1)
- moved X102 51.1 mm to (213.9, 168.2)
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Connections:
- net /D+ renamed /Project Architecture/Main/D+
- net /D- renamed /Project Architecture/Main/D-
- net /D_{2}+ renamed /Project Architecture/Main/D_{2}+
- net /D_{2}- renamed /Project Architecture/Main/D_{2}-
Other:
- board text added: "${ASSEMBLY_NOTES}"
- board text added: "${FABRICATION_NOTES}"
- board text added: "0.01mm"
- board text added: "0.035mm (1oz)"
- board text added: "1.51mm"
- board text added: "Bottom View"
- board text added: "Components"
- board text added: "Copper"
- board text added: "Core"
- board text added: "Dielectric"
- board text added: "Drill Table"
- board text added: "GBR"
- board text added: "Gerber"
- board text added: "Impedance Table"
- board text added: "Layer"
- board text added: "Layer Stack Legend"
- board text added: "Legend"
- board text added: "Note: external layer thicknesses are specified after plating"
- board text added: "Paste Mask"
- board text added: "Signal"
- board text added: "Solder Mask"
- board text added: "Thickness"
- board text added: "Top View"
- board text added: "Total thickness: 1.6mm"
- board text added: "Type"
- board text removed: "0"
- board text removed: "0 mm"
- board text removed: "0,01 mm"
- board text removed: "0,02"
- board text removed: "0,035 mm"
- board text removed: "0,1250 mm / 0,1250 mm"
- board text removed: "0,196 mm"
- board text removed: "0,2500 mm"
- board text removed: "0,43 mm"
- board text removed: "1"
- board text removed: "1,5260 mm"
- board text removed: "3,3"
- board text removed: "4"
- board text removed: "4,5"
- board text removed: "80,0000 mm x 48,0000 mm"
- board text removed: "Abmessungen der Platine:"
- board text removed: "Blue"
- board text removed: "Bottom Silk Screen"
- board text removed: "Bottom Solder Mask"
- board text removed: "Bottom Solder Paste"
- board text removed: "Castellated Pads:"
- board text removed: "Dicke (mm)"
- board text removed: "Dielektrikum"
- board text removed: "Epsilon R"
- board text removed: "FR4 natural"
- board text removed: "Farbe"
- board text removed: "HAL SnPb"
- board text removed: "Impedanzkontrolle:"
- board text removed: "Inner1"
- board text removed: "Inner2"
- board text removed: "Kupferlagenanzahl:"
- board text removed: "Kupferoberfläche:"
- board text removed: "Lagenname"
- board text removed: "Metallisierte Platinenkante:"
- board text removed: "Min Leiterbahn/abstand:"
- board text removed: "Min Lochdurchmesser:"
- board text removed: "Nein"
- board text removed: "Not specified"
- board text removed: "PLATINEN-EIGENSCHAFTEN"
- board text removed: "Platinen-Dicke:"
- board text removed: "Randsteckverbinder:"
- board text removed: "Tangens des Verlustwinkels"
- board text removed: "Top Silk Screen"
- board text removed: "Top Solder Mask"
- board text removed: "Top Solder Paste"
- board text removed: "Typ"
- board text removed: "White"
- board text removed: "copper"
- board text removed: "core"
- board text removed: "prepreg"
