File: hardware/ZSWatch-Dock.kicad_sch (KiCad schematic)
At the start: 67 parts, among them IC101 TLV70218_SOT23-5, IC102 USBLC6-2P6, IC103 FT230XQ, IC104 MIC5219-3.3YM5, IC105 NL3V4T244MU2TAG-Q, IC106 USBLC6-2P6, IC107 USB2512BT, IC108 USBLC6-2P6, IC109 MIC2026-1xM, J101 Jumper, J102 Voltage, Q101 BSH205G2AR, SW101 Charge, X101 Debug, X102 UART, X103 Host, X104 Device, X105 Current, Y101 24 MHz

Commit message: Issue #42
Parts:
- removed C101, C103, C104, C105, C106, C107, C109, C114, C115, C116, C117, C118, C119: 100n, Capacitor_SMD:C_0603_1608Metric, symbol Device:C_Small
- removed C102, C111: 2u2, Capacitor_SMD:C_0603_1608Metric, symbol Device:C_Small
- removed C108: 470p, Capacitor_SMD:C_0603_1608Metric, symbol Device:C_Small
- removed C110: 1u, Capacitor_SMD:C_0603_1608Metric, symbol Device:C_Small
- removed C112, C113: 18p, Capacitor_SMD:C_0603_1608Metric, symbol Device:C_Small
- removed D101, D102: ESD5Zxx, Diode_SMD:D_SOD-523, symbol Diode:ESD5Zxx
- removed D103: USB, LED_SMD:LED_0603_1608Metric, symbol Device:LED
- removed D104: Charge, LED_SMD:LED_0603_1608Metric, symbol Device:LED
- removed IC101: TLV70218_SOT23-5, Package_TO_SOT_SMD:SOT-23-5, symbol Regulator_Linear:TLV70218_SOT23-5
- removed IC102, IC106, IC108: USBLC6-2P6, Package_TO_SOT_SMD:SOT-666, symbol Power_Protection:USBLC6-2P6
- removed IC103: FT230XQ, Package_DFN_QFN:QFN-16-1EP_4x4mm_P0.65mm_EP2.1x2.1mm, symbol Interface_USB:FT230XQ
- removed IC104: MIC5219-3.3YM5, Package_TO_SOT_SMD:SOT-23-5, symbol Regulator_Linear:MIC5219-3.3YM5
- removed IC105: NL3V4T244MU2TAG-Q, Package_SO:TSSOP-14_4.4x5mm_P0.65mm, symbol ON Semiconductor:NL3V4T244 (TSSOP14)
- removed IC107: USB2512BT, Package_DFN_QFN:QFN-36-1EP_6x6mm_P0.5mm_EP3.7x3.7mm, symbol Microchip_Kampi:USB2512BT
- removed IC109: MIC2026-1xM, Package_SO:SOIC-8_3.9x4.9mm_P1.27mm, symbol Power_Management:MIC2026-1xM
- removed J101: Jumper, symbol Misc:Jumper
- removed J102: Voltage, Connector_PinHeader_2.54mm:PinHeader_1x03_P2.54mm_Vertical, symbol Connector_Generic:Conn_01x03
- removed Q101: BSH205G2AR, Package_TO_SOT_SMD:SOT-23, symbol Nexperia:BSH205G2AR
- removed R101, R102, R108, R110, R111, R112, R117, R119: 100k, Resistor_SMD:R_0603_1608Metric, symbol Device:R_Small
- removed R103, R104, R115: 0R, Resistor_SMD:R_0805_2012Metric, symbol Device:R_Small
- removed R105, R106, R113, R114: 5k1, Resistor_SMD:R_0603_1608Metric, symbol Device:R_Small
- removed R107: 3k3, Resistor_SMD:R_0603_1608Metric, symbol Device:R_Small
- removed R109: 1M, Resistor_SMD:R_0603_1608Metric, symbol Device:R_Small
- removed R116: 12k / 1%, Resistor_SMD:R_0603_1608Metric, symbol Device:R_Small
- removed R118: 620R, Resistor_SMD:R_0603_1608Metric, symbol Device:R_Small
- removed R120, R121: 22R, Resistor_SMD:R_0603_1608Metric, symbol Device:R_Small
- removed S101: Reset, Wuerth:WS-TASV-6x6, symbol Switch:SW_Push
- removed SB101: Resetn, Jumper:SolderJumper-2_P1.3mm_Open_RoundedPad1.0x1.5mm, symbol Jumper:SolderJumper_2_Open
- removed SB102: SWDCLK, Jumper:SolderJumper-2_P1.3mm_Open_RoundedPad1.0x1.5mm, symbol Jumper:SolderJumper_2_Open
- removed SB103: SWDIO, Jumper:SolderJumper-2_P1.3mm_Open_RoundedPad1.0x1.5mm, symbol Jumper:SolderJumper_2_Open
- removed SW101: Charge, Button_Switch_SMD:SW_SPDT_PCM12, symbol Switch:SW_DPDT_x2
- removed X101: Debug, Samtec:SHF-105-01-L-D-SM-TR, symbol Connector:Conn_ARM_JTAG_SWD_10
- removed X102: UART, Connector_PinHeader_2.54mm:PinHeader_1x03_P2.54mm_Vertical, symbol Connector_Generic:Conn_01x03
- removed X103: Host, Connector_USB:USB_C_Receptacle_Amphenol_12401610E4-2A, symbol Connector:USB_C_Receptacle
- removed X104: Device, Connector_USB:USB_C_Receptacle_Amphenol_12401610E4-2A, symbol Connector:USB_C_Receptacle
- removed X105: Current, Connector_PinHeader_2.54mm:PinHeader_1x02_P2.54mm_Horizontal, symbol Connector_Generic:Conn_01x02
- removed Y101: 24 MHz, Crystal:Crystal_SMD_Abracon_ABM8G-4Pin_3.2x2.5mm, symbol Device:Crystal_GND24
Connections:
- no-connect marks 22 -> 0
Other:
- added sheet Block Diagram (Block Diagram.kicad_sch)
- added sheet Power - Sequencing (Power - Sequencing.kicad_sch)
- added sheet Project Architecture (Project Architecture.kicad_sch)
- added sheet Revision History (Revision History.kicad_sch)
- note added: "${BOARD_NAME}"
- note added: "${RELEASE_DATE_NUM}"
- note added: "${SHEET_NAME_10}"
- note added: "${SHEET_NAME_11}"
- note added: "${SHEET_NAME_12}"
- note added: "${SHEET_NAME_13}"
- note added: "${SHEET_NAME_14}"
- note added: "${SHEET_NAME_15}"
- note added: "${SHEET_NAME_16}"
- note added: "${SHEET_NAME_17}"
- note added: "${SHEET_NAME_18}"
- note added: "${SHEET_NAME_19}"
- note added: "${SHEET_NAME_1}"
- note added: "${SHEET_NAME_20}"
- note added: "${SHEET_NAME_21}"
- note added: "${SHEET_NAME_22}"
- note added: "${SHEET_NAME_23}"
- note added: "${SHEET_NAME_24}"
- note added: "${SHEET_NAME_25}"
- note added: "${SHEET_NAME_26}"
- note added: "${SHEET_NAME_27}"
- note added: "${SHEET_NAME_28}"
- note added: "${SHEET_NAME_29}"
- note added: "${SHEET_NAME_2}"
- note added: "${SHEET_NAME_30}"
- note added: "${SHEET_NAME_31}"
- note added: "${SHEET_NAME_32}"
- note added: "${SHEET_NAME_33}"
- note added: "${SHEET_NAME_34}"
- note added: "${SHEET_NAME_35}"
- note added: "${SHEET_NAME_36}"
- note added: "${SHEET_NAME_37}"
- note added: "${SHEET_NAME_38}"
- note added: "${SHEET_NAME_39}"
- note added: "${SHEET_NAME_3}"
- note added: "${SHEET_NAME_40}"
- note added: "${SHEET_NAME_4}"
- note added: "${SHEET_NAME_5}"
- note added: "${SHEET_NAME_6}"
- note added: "${SHEET_NAME_7}"
- note added: "${SHEET_NAME_8}"
- note added: "${SHEET_NAME_9}"
- note added: "1"
- note added: "10"
- note added: "11"
- note added: "12"
- note added: "13"
- note added: "14"
- note added: "15"
- note added: "16"
- note added: "17"
- note added: "18"
- note added: "19"
- note added: "2"
- note added: "20"
- note added: "21"
- note added: "22"
- note added: "23"
- note added: "24"
- note added: "25"
- note added: "26"
- note added: "27"
- note added: "28"
- note added: "29"
- note added: "3"
- note added: "30"
- note added: "31"
- note added: "32"
- note added: "33"
- note added: "34"
- note added: "35"
- note added: "36"
- note added: "37"
- note added: "38"
- note added: "39"
- note added: "4"
- note added: "40"
- note added: "5"
- note added: "6"
- note added: "7"
- note added: "8"
- note added: "9"
- note added: "BOTTOM VIEW"
- note added: "CHECKED - There shouldn't be any mistakes. Contact the engineer if you find any."
- note added: "Comment"
- note added: "DESIGN CONSIDERATIONS"
- note added: "DRAFT - Very early stage of schematic, ignore details."
- note added: "Date: ${RELEASE_DATE}"
- note added: "Index"
- note added: "NOTES"
- note added: "Not fitted components are marked as"
- note added: "PRELIMINARY - Close to final schematic."
- note added: "Page"
- note added: "RELEASED - A board with this schematic has been sent to production."
- note added: "Rev ${REVISION}"
- note added: "TOP VIEW"
- note added: "Variant: ${VARIANT}"
- note removed: "1V8 Regulator"
- note removed: "1V8 domain"
- note removed: "3V3 Regulator"
- note removed: "90 Ohm ± 15%"
- note removed: "Active-high for MIC20x6-1"
- note removed: "Active-low output with Pull-Up on USB hub"
- note removed: "Configuration: - All ports are non-removable (REM0 = low and REM1 = high) - LED is active low (REM0 = low and REM1 = high) - Strap options enabled (CFG_SEL0 and CFG_SEL1 = low) - Self-powered operation enabled (CFG_SEL0 and CFG_SEL1 = low) - Individual power switching enabled (CFG_SEL0 and CFG_SEL1 = low) - Individual over-current sensing enabled (CFG_SEL0 and CFG_SEL1 = low) - Enable battery opt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"
- note removed: "FT230X"
- note removed: "Low ESR capacitors"
- note removed: "Reset"
- note removed: "SWD"
- note removed: "USB (To Client/ZSWatch)"
- note removed: "USB (To Host/Computer)"
- note removed: "USB <-> UART"
- note removed: "USB251xB contains an internal 1M resistor"
- note removed: "ZSWatch"
- company: github.com/ZSWatch/Dock-HW -> ${COMPANY}
- title: ZSWatch Dock v2 -> Dock-HW
